File: signalprocessing/signalprocessing.kicad_sch (KiCad schematic)
At the start: 40 parts, among them IC1 MCP6022-I_P, IC2 NJU7043D, J1 MJ-8435, J10 22-23-2021, J2 22-23-2021, J3 22-23-2021, J4 22-23-2021, J5 22-23-2021, J6 22-23-2021, J7 MJ-8435, J8 22-23-2021, J9 22-23-2021, U1 Nucleo64-F446

Commit message: 4
Parts:
- added TP2, TP4: TestPoint, TestPoint:TestPoint_Loop_D2.50mm_Drill1.0mm, symbol Connector:TestPoint
- C1, C8: value 0.1μ -> 1μ
- C11: footprint Capacitor_THT:C_Disc_D4.7mm_W2.5mm_P5.00mm -> Capacitor_THT:CP_Radial_D5.0mm_P2.50mm
- C6: footprint RScomponents:ECQUBAF332MA -> Capacitor_THT:C_Rect_L7.0mm_W2.0mm_P5.00mm
- C7: footprint RScomponents:ECQUBAF332MA -> Capacitor_THT:C_Rect_L7.0mm_W3.5mm_P5.00mm
- RV1: footprint RScomponents:RK097221004C -> RScomponents:RK09712200HA
- renumbered J7 to J2, J2 to JP1, J3 to JP11, J5 to JP12, J10 to JP13, J8 to JP14, J4 to JP2, J9 to JP3, J6 to JP4, TP2 to TP3
Connections:
- net GND: now also TP2.1, TP4.1
Other:
- note added: "1"
- note added: "2"
- note added: "3"
- note added: "4"

Commit message: 2
Parts:
- C10, C5: footprint Capacitor_THT:C_Disc_D4.7mm_W2.5mm_P5.00mm -> Capacitor_THT:C_Disc_D3.8mm_W2.6mm_P2.50mm
Connections:
- net R13: now reaches C8.2, JP3.1
- net R13: now also RV1.R13 (3); no longer RV1.R11 (1)
- net R11: now reaches C4.2, C9.2, R1.2, R11.1, R2.1, R7.2, R8.1
- net R11: now also RV1.R11 (1); no longer RV1.R13 (3)
Changed lines of the file:
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@@
   (junction (at 171.45 109.22) (diameter 0) (color 0 0 0 0)
   )
+  (junction (at 231.14 95.25) (diameter 0) (color 0 0 0 0)
+  )
+  (junction (at 209.55 64.77) (diameter 0) (color 0 0 0 0)
+  )
+  (junction (at 102.87 76.2) (diameter 0) (color 0 0 0 0)
+  )
+  (junction (at 222.25 81.28) (diameter 0) (color 0 0 0 0)
+  )
+  (junction (at 80.01 114.3) (diameter 0) (color 0 0 0 0)
+  )
+  (junction (at 251.46 82.55) (diameter 0) (color 0 0 0 0)
+  )
+  (junction (at 63.5 85.09) (diameter 0) (color 0 0 0 0)
+  )
+  (junction (at 196.85 64.77) (diameter 0) (color 0 0 0 0)
+  )
+  (junction (at 62.23 111.76) (diameter 0) (color 0 0 0 0)
+  )
   (junction (at 176.53 80.01) (diameter 0) (color 0 0 0 0)
-  )
-  (junction (at 231.14 95.25) (diameter 0) (color 0 0 0 0)
-  )
-  (junction (at 209.55 64.77) (diameter 0) (color 0 0 0 0)
-  )
-  (junction (at 102.87 76.2) (diameter 0) (color 0 0 0 0)
-  )
-  (junction (at 222.25 81.28) (diameter 0) (color 0 0 0 0)
-  )
-  (junction (at 80.01 114.3) (diameter 0) (color 0 0 0 0)
-  )
-  (junction (at 251.46 82.55) (diameter 0) (color 0 0 0 0)
-  )
-  (junction (at 63.5 85.09) (diameter 0) (color 0 0 0 0)
-  )
-  (junction (at 196.85 64.77) (diameter 0) (color 0 0 0 0)
-  )
-  (junction (at 62.23 111.76) (diameter 0) (color 0 0 0 0)
   )
   (no_connect (at 233.68 85.09))
@@
     (effects (font (size 1.27 1.27)) (justify left bottom))
   )
+  (label "R11" (at 176.53 90.17 0)
+    (effects (font (size 1.27 1.27)) (justify left bottom))
+  )
+  (label "R13" (at 176.53 76.2 0)
+    (effects (font (size 1.27 1.27)) (justify left bottom))
+  )
   (symbol (lib_id "Device:R") (at 69.85 114.3 90) (unit 1)
     (in_bom yes) (on_board yes)
@@
     (property "Reference" "C10" (id 0) (at 199.39 52.07 90))
     (property "Value" "0.1μ" (id 1) (at 204.47 53.34 90))
-    (property "Footprint" "Capacitor_THT:C_Disc_D4.7mm_W2.5mm_P5.00mm" (id 2) (at 204.47 54.9148 0)
+    (property "Footprint" "Capacitor_THT:C_Disc_D3.8mm_W2.6mm_P2.50mm" (id 2) (at 204.47 54.9148 0)
       (effects (font (size 1.27 1.27)) hide)
     )
@@
     (pin "2")
   )
-  (symbol (lib_id "Device:R_Potentiometer") (at 176.53 83.82 0) (unit 1)
-    (in_bom yes) (on_board yes)
-    (property "Reference" "RV1" (id 0) (at 176.53 78.74 0)
+  (symbol (lib_id "Device:R_Potentiometer") (at 176.53 83.82 0) (mirror x) (unit 1)
+    (in_bom yes) (on_board yes)
+    (property "Reference" "RV1" (id 0) (at 181.61 80.01 0)
       (effects (font (size 1.27 1.27)) (justify right))
     )
-    (property "Value" "R_Potentiometer" (id 1) (at 185.42 66.04 0)
+    (property "Value" "R_Potentiometer" (id 1) (at 185.42 101.6 0)
       (effects (font (size 1.27 1.27)) (justify right))
     )
-    (property "Footprint" "RScomponents:RK09712200HA" (id 2) (at 179.07 91.44 0)
+    (property "Footprint" "RScomponents:RK09712200HA" (id 2) (at 179.07 76.2 0)
       (effects (font (size 1.27 1.27)) hide)
     )
@@
     (property "Reference" "C5" (id 0) (at 107.95 62.23 90))
     (property "Value" "0.1μ" (id 1) (at 109.22 64.77 90))
-    (property "Footprint" "Capacitor_THT:C_Disc_D4.7mm_W2.5mm_P5.00mm" (id 2) (at 104.14 69.5452 0)
+    (property "Footprint" "Capacitor_THT:C_Disc_D3.8mm_W2.6mm_P2.50mm" (id 2) (at 104.14 69.5452 0)
       (effects (font (size 1.27 1.27)) hide)
     )
@@
     )
     (path "/dd97b578-62b8-46ea-b6db-aa022cf0712b"
-      (reference "C5") (unit 1) (value "0.1μ") (footprint "Capacitor_THT:C_Disc_D4.7mm_W2.5mm_P5.00mm")
+      (reference "C5") (unit 1) (value "0.1μ") (footprint "Capacitor_THT:C_Disc_D3.8mm_W2.6mm_P2.50mm")
     )
     (path "/4ba434e6-1c98-4b73-8536-32f634dc2cc7"
@@
     )
     (path "/2b87babf-3ede-4677-8599-584b848f3fdf"
-      (reference "C10") (unit 1) (value "0.1μ") (footprint "Capacitor_THT:C_Disc_D4.7mm_W2.5mm_P5.00mm")
+      (reference "C10") (unit 1) (value "0.1μ") (footprint "Capacitor_THT:C_Disc_D3.8mm_W2.6mm_P2.50mm")
     )
     (path "/f0a25887-5f46-4352-b61b-1723c84fd18a"
