File: signalprocessing/signalprocessing.kicad_pcb (KiCad board)
At the start: 2 copper layers, 54 x 99.8 mm, 212 parts, among them IC1 MCP6022-I_P, IC2 NJU7043D, J1 MJ-8435, J10 22-23-2021, J2 MJ-8435, J3 22-23-2021, J5 22-23-2021, J6 22-23-2021, U1 Nucleo64-F446

Commit message: 4
Parts:
- added G***: LOGO, Interface_Library:logo2, F.Cu at (80.5, 135.4)
- added TP2: TestPoint, TestPoint:TestPoint_Loop_D2.50mm_Drill1.0mm, F.Cu at (107.3, 88.3)
- added TP4: TestPoint, TestPoint:TestPoint_Loop_D2.50mm_Drill1.0mm, F.Cu at (101.6, 88.3)
- C11: footprint Capacitor_THT:C_Disc_D4.7mm_W2.5mm_P5.00mm -> Capacitor_THT:CP_Radial_D5.0mm_P2.50mm
- C6: footprint Capacitor_THT:C_Rect_L4.0mm_W2.5mm_P2.50mm -> Capacitor_THT:C_Rect_L7.0mm_W2.0mm_P5.00mm
- C7: footprint Capacitor_THT:C_Rect_L4.0mm_W2.5mm_P2.50mm -> Capacitor_THT:C_Rect_L7.0mm_W3.5mm_P5.00mm
- RV1 (x2): footprint RScomponents:RK097221004C -> RScomponents:RK09712200HA
- moved C11 1.81 mm to (87.7, 128.3)
- moved C6 1.46 mm to (109.3, 97.2)
- moved C7 1.29 mm to (109.3, 93.3)
- moved JP1 1.27 mm to (88.9, 142.2)
- moved JP11 1.27 mm to (86.0, 139.7)
- moved R11 0.64 mm to (106.0, 103.5)
- moved C8 0.63 mm to (90.2, 103.5)
- moved J1 0.51 mm to (122.2, 76.1)
- moved J2 0.51 mm to (87.4, 76.1)
- renumbered J3 to JP11, J5 to JP12, J10 to JP13, JP2 to JP14, JP4 to JP2, J6 to JP4, TP2 to TP3
Connections:
- C8 pad 2: Net-(C9-Pad2) -> Net-(C8-Pad2)
- JP3 pad 1: Net-(C9-Pad2) -> Net-(C8-Pad2)
Routing:
- net Net-(C8-Pad2): track 0.00 -> 82.3 mm
- net Net-(C9-Pad2): track 81.0 -> 0.00 mm
- net Net-(JP1-Pad1): track 30.5 -> 27.7 mm
- net +5V: track 39.5 -> 41.3 mm
- net Net-(IC2-Pad1): track 34.9 -> 33.2 mm
- net Net-(C7-Pad1): track 7.17 -> 8.46 mm
- net Net-(JP1-Pad2): track 31.3 -> 32.5 mm
- net Net-(JP11-Pad2): track 36.5 -> 35.5 mm
Other:
- outline, holes or cut-outs redrawn
- board text added: "1"
- board text added: "2"
- board text added: "3"
- board text added: "4"
- board text added: "https://interface.cqpub.co.jp/"
- board text added: "ディジタル信号処理"

Commit message: 2
Parts:
- C1, C8: value 0.1μ -> 1μ
- C10, C5: footprint Capacitor_THT:C_Disc_D4.7mm_W2.5mm_P5.00mm -> Capacitor_THT:C_Disc_D3.8mm_W2.6mm_P2.50mm
- moved C10 2.77 mm to (96.2, 127.0)
- moved C5 2.39 mm to (123.7, 133.3)
- moved C7 2.33 mm to (107.2, 94.5)
- moved C6 2.22 mm to (107.2, 98.0)
- moved TP2 1.66 mm to (107.4, 89.9)
- moved TP4 1.65 mm to (101.6, 89.9)
Connections:
- C4 pad 2: Net-(C4-Pad2) -> /R11
- C8 pad 2: Net-(C8-Pad2) -> /R13
- C9 pad 2: Net-(C4-Pad2) -> /R11
- JP3 pad 1: Net-(C8-Pad2) -> /R13
- R1 pad 2: Net-(C4-Pad2) -> /R11
- R11 pad 1: Net-(C4-Pad2) -> /R11
- R2 pad 1: Net-(C4-Pad2) -> /R11
- R7 pad 2: Net-(C4-Pad2) -> /R11
- R8 pad 1: Net-(C4-Pad2) -> /R11
- REF**9 pad 1: (no net) -> GND
- RV1 pad R13: Net-(C4-Pad2) -> /R13 (x2)
- RV1 pad R21: (no net) -> /R11
- RV1 pad R22: (no net) -> Net-(IC2-Pad5)
- RV1 pad R23: (no net) -> /R13
Routing:
- net /R11: track 0.00 -> 129.9 mm
- net Net-(C4-Pad2): track 114.9 -> 0.00 mm
- net Net-(C8-Pad2): track 82.3 -> 0.00 mm
- net /R13: track 0.00 -> 81.4 mm
- net GND: track 0.00 -> 5.79 mm
- net Net-(IC2-Pad5): track 75.2 -> 72.4 mm, vias 1 -> 0
- net Net-(C7-Pad1): track 8.46 -> 5.98 mm
- net Net-(C6-Pad1): track 12.0 -> 9.75 mm
- net Net-(IC1-Pad1): track 29.3 -> 30.5 mm
- net Net-(C1-Pad2): track 47.5 -> 48.2 mm
Other:
- outline, holes or cut-outs redrawn
- board text added: "GND"

Commit message: 3
Parts:
- C10, C5: footprint Capacitor_THT:C_Disc_D3.8mm_W2.6mm_P2.50mm -> Capacitor_THT:C_Disc_D4.3mm_W1.9mm_P5.00mm
- moved C11 2.85 mm to (87.1, 125.5), turned to -90 degrees
- moved C5 2.55 mm to (121.3, 132.5)
- moved C10 0.87 mm to (97.1, 127.0)
Connections:
- C11 pad 1: GND -> +5V
- C11 pad 2: +5V -> GND
Routing:
- net +5V: track 41.3 -> 39.1 mm
- net Net-(IC1-Pad1): track 30.5 -> 31.7 mm
